Commit message: fix plannar and hand_controller bug

File: install/panda_description/share/panda_description/urdf/panda_description_gazebo.xacro (robot description, xacro)
@@ -364,14 +364,24 @@
           <state_interface name="velocity"/>
       </joint>
-      <joint name="panda_joint8">
-          <command_interface name="position">
-              <param name="min">-1</param>
-              <param name="max">1</param>
-          </command_interface>
-          <state_interface name="position">
-              <param name="initial_value">0.0</param>
-          </state_interface>
-          <state_interface name="velocity"/>
-      </joint>
+        <joint name="panda_finger_joint1">
+            <command_interface name="position" />
+            <state_interface name="position">
+                <param name="initial_value">0.0</param>
+            </state_interface>
+            <state_interface name="velocity">
+                <param name="initial_value">0.0</param>
+            </state_interface>
+        </joint>
+        <joint name="panda_finger_joint2">
+            <param name="mimic">panda_finger_joint1</param>
+            <param name="multiplier">1</param>
+            <command_interface name="position" />
+            <state_interface name="position">
+                <param name="initial_value">0.0</param>
+            </state_interface>
+            <state_interface name="velocity">
+                <param name="initial_value">0.0</param>
+            </state_interface>
+        </joint>
   </ros2_control>
   <!-- gazebo -->

File: install/panda_moveit_config/share/panda_moveit_config/config/panda_ros2_control.xacro (robot description, xacro)
@@ -3,5 +3,5 @@
     <xacro:macro name="panda_ros2_control" params="initial_positions_file ros2_control_hardware_type">
         <xacro:property name="initial_positions" value="${xacro.load_yaml(initial_positions_file)['initial_positions']}"/>
-        <ros2_control name="mock" type="system"> <!--GazeboSimSystem-->>
+        <ros2_control name="mock" type="system"> <!--GazeboSimSystem-->
             <hardware>
                 <xacro:if value="${ros2_control_hardware_type == 'mock_components'}">
@@ -84,5 +84,5 @@
                 <command_interface name="position"/>
                 <state_interface name="position">
-                  <param name="initial_value">0.0</param>
+                  <param name="initial_value">${initial_positions['panda_finger_joint1']}</param>
                 </state_interface>
                 <state_interface name="velocity">
@@ -91,10 +91,11 @@
             </joint>
             <joint name="panda_finger_joint2">
-                <command_interface name="position"/>
+                <param name="mimic">panda_finger_joint1</param>
+                <param name="multiplier">1</param>
                 <state_interface name="position">
                   <param name="initial_value">0.0</param>
                 </state_interface>
                 <state_interface name="velocity">
-                  <param name="initial_value">0.0</param>
+                    <param name="initial_value">0.0</param>
                 </state_interface>
             </joint>
