Commit message: add camera

File: install/panda_description/share/panda_description/urdf/camera/camera.xacro (robot description, xacro)
@@ -11,10 +11,10 @@
 	  <visual>
 		<geometry>
-		  <mesh filename="package://panda_description/meshes/visual/camera.dae"/>
+		  <mesh filename="$(find panda_description)/meshes/visual/camera.dae"/>
 		</geometry>
 	  </visual>
 	  <collision>
 		<geometry>
-		  <mesh filename="package://panda_description/meshes/collision/camera.stl"/>
+		  <mesh filename="$(find panda_description)/meshes/collision/camera.stl"/>
 		</geometry>
 	  </collision>
@@ -26,3 +26,32 @@
 	</link>
   </xacro:macro>
+  <gazebo reference="camera_link">
+        <!-- <material>Gazebo/Red</material> -->
+        <sensor name="camera" type="camera">
+            <pose> 0 0 0 0 0 0 </pose>
+            <visualize>true</visualize>
+            <update_rate>10</update_rate>
+            <camera>
+                <horizontal_fov>1.089</horizontal_fov>
+                <image>
+                    <format>R8G8B8</format>
+                    <width>640</width>
+                    <height>480</height>
+                </image>
+                <clip>
+                    <near>0.05</near>
+                    <far>8.0</far>
+                </clip>
+            </camera>
+			<plugin name="camera_controller" filename="libgazebo_ros_camera.so">
+				<alwaysOn>true</alwaysOn>
+				<updateRate>0.0</updateRate>
+				<cameraName>panda/camera1</cameraName>
+				<imageTopicName>image_raw</imageTopicName>
+				<cameraInfoTopicName>camera_info</cameraInfoTopicName>
+				<frameName>camera_link</frameName>
+				<hackBaseline>0.07</hackBaseline>
+			</plugin>
+        </sensor>
+    </gazebo >
 </robot>

File: install/panda_description/share/panda_description/urdf/panda_description_gazebo.xacro (robot description, xacro)
@@ -290,4 +290,11 @@
   </joint>
   <link name="random"/>
+  <!-- Camera -->
+  <xacro:include filename="$(find panda_description)/urdf/camera/camera.xacro"/>
+  <xacro:camera_v0 parent="panda_link0">
+   <origin xyz="0.2 0.6 0.7" rpy="0 1.57 0"/>
+  </xacro:camera_v0>
+  <xacro:camera_gazebo_v0/>
+  <!-- Camera -->
   <ros2_control name="GazeboSystem" type="system">
       <hardware>
@@ -385,5 +392,5 @@
         </joint>
   </ros2_control>
-  <!-- gazebo -->
+  <!-- gazebo reference="camera_link"-->
   <gazebo>
     <plugin name="gazebo_ros2_control" filename="libgazebo_ros2_control.so">
@@ -391,4 +398,29 @@
         <robot_param_node>robot_state_publisher</robot_param_node>
     </plugin>
+    <!-- <plugin name="camera_controller" filename="libgazebo_ros_camera.so">
+        <alwaysOn>true</alwaysOn>
+        <updateRate>0.0</updateRate>
+        <cameraName>panda/camera1</cameraName>
+        <imageTopicName>image_raw</imageTopicName>
+        <cameraInfoTopicName>camera_info</cameraInfoTopicName>
+        <frameName>camera_link</frameName>
+        <hackBaseline>0.07</hackBaseline>
+    </plugin> -->
   </gazebo>
+  <!-- <gazebo reference="camera_link">
+    <plugin name="camera_controller" filename="libgazebo_ros_camera.so">
+        <alwaysOn>true</alwaysOn>
+        <updateRate>0.0</updateRate>
+        <cameraName>panda/camera1</cameraName>
+        <imageTopicName>image_raw</imageTopicName>
+        <cameraInfoTopicName>camera_info</cameraInfoTopicName>
+        <frameName>camera_link</frameName>
+        <hackBaseline>0.07</hackBaseline>
+        <distortionK1>0.0</distortionK1>
+        <distortionK2>0.0</distortionK2>
+        <distortionK3>0.0</distortionK3>
+        <distortionT1>0.0</distortionT1>
+        <distortionT2>0.0</distortionT2>
+      </plugin>
+  </gazebo> -->
 </robot>

File: install/panda_moveit_config/share/panda_moveit_config/config/panda.urdf.xacro (robot description, xacro)
@@ -8,10 +8,10 @@
     <xacro:include filename="$(find panda_description)/urdf/panda_description.xacro" />
     <!-- <xacro:include filename="$(find panda_description)/urdf/panda_description_gazebo.xacro" /> -->
-    <!-- <xacro:include filename="$(find panda_description)/urdf/camera/camera.xacro"/> -->
+      <xacro:include filename="$(find panda_description)/urdf/camera/camera.xacro"/>
     <!-- Camera -->
-    <!-- <xacro:camera_v0 parent="panda_link0">
+    <xacro:camera_v0 parent="panda_link0">
 	    <origin xyz="0.2 0.6 0.7" rpy="0 ${PI/2} 0"/>
     </xacro:camera_v0>
-    <xacro:camera_gazebo_v0/> -->
+    <!-- <xacro:camera_gazebo_v0/> -->
     <!-- controllers for gazebo -->
     <!-- <xacro:include filename="panda.gazebo_ros2_control.xacro" />  -->
@@ -25,25 +25,18 @@
         <robot_param_node>robot_state_publisher</robot_param_node>
       </plugin>
+      <plugin name="camera_controller" filename="libgazebo_ros_camera.so">
+        <alwaysOn>true</alwaysOn>
+        <updateRate>0.0</updateRate>
+        <cameraName>rrbot/camera1</cameraName>
+        <imageTopicName>image_raw</imageTopicName>
+        <cameraInfoTopicName>camera_info</cameraInfoTopicName>
+        <frameName>camera_link</frameName>
+        <hackBaseline>0.07</hackBaseline>
+        <distortionK1>0.0</distortionK1>
+        <distortionK2>0.0</distortionK2>
+        <distortionK3>0.0</distortionK3>
+        <distortionT1>0.0</distortionT1>
+        <distortionT2>0.0</distortionT2>
+      </plugin>
     </gazebo>
-  <!-- <gazebo>
-    <plugin
-        filename="gz_ros2_control-system"
-        name="gz_ros2_control::GazeboSimROS2ControlPlugin">
-        <parameters>$(find panda_moveit_config)/config/ros2_controllers.yaml</parameters>
-    </plugin>
-    <plugin
-        filename="gz-sim-joint-state-publisher-system"
-        name="gz::sim::systems::JointStatePublisher">
-    </plugin>
-    <plugin
-        filename="gz-sim-pose-publisher-system"
-        name="gz::sim::systems::PosePublisher">
-        <publish_link_pose>true</publish_link_pose>
-        <use_pose_vector_msg>true</use_pose_vector_msg>
-        <publish_nested_model_pose>true</publish_nested_model_pose>
-    </plugin>
-    <plugin filename="ignition-gazebo-sensors-system" name="ignition::gazebo::systems::Sensors">
-      <render_engine>ogre2</render_engine>
-    </plugin>
-  </gazebo> -->
 </robot>

File: src/panda_description/urdf/panda_description_gazebo.xacro (robot description, xacro)
@@ -290,4 +290,11 @@
   </joint>
   <link name="random"/>
+  <!-- Camera -->
+  <xacro:include filename="$(find panda_description)/urdf/camera/camera.xacro"/>
+  <xacro:camera_v0 parent="panda_link0">
+   <origin xyz="0.2 0.6 0.7" rpy="0 1.57 0"/>
+  </xacro:camera_v0>
+  <xacro:camera_gazebo_v0/>
+  <!-- Camera -->
   <ros2_control name="GazeboSystem" type="system">
       <hardware>
@@ -385,5 +392,4 @@
         </joint>
   </ros2_control>
-  <!-- gazebo -->
   <gazebo>
     <plugin name="gazebo_ros2_control" filename="libgazebo_ros2_control.so">
